File: esp32_relay.kicad_pcb (KiCad board)
At the start: 2 copper layers, 212.1 x 110.4 mm, 106 parts, among them J1 LCD, J10 Screw_Terminal_01x03, J11 Screw_Terminal_01x02, J12 Screw_Terminal_01x02, J13 Screw_Terminal_01x02, J14 Screw_Terminal_01x04, J15 Screw_Terminal_01x03, J16 Screw_Terminal_01x03, J17 Screw_Terminal_01x03, J18 Screw_Terminal_01x03, J19 Conn_01x02_Female, J20 Conn_01x02_Female, J21 Screw_Terminal_01x02, J22 Screw_Terminal_01x02, J23 Screw_Terminal_01x02, J24 Power, J25 MT1, J26 MT4, J27 MT2, J28 MT3, J3 Conn_01x03, J4 Conn_01x02_Female, J5 Conn_01x02_Female, J6 Screw_Terminal_01x03, J7 Screw_Terminal_01x03, J8 Screw_Terminal_01x03, J9 Screw_Terminal_01x03, K1 Relay, K2 Relay, K3 Relay, K4 Relay, K5 Relay, K6 Relay, K7 Relay, K8 Relay, SW1 Boot, U1 LM2596S-5, U10 PC817, U11 PC817, U12 PC817, U13 PC817, U14 PC817, U15 MAX485E, U2 AMS1117-3.3, U3 ESP32-WROOM-32U, U4 L298N, U5 L298N, U6 PCF8574ATS, U7 PC817, U8 PC817, U9 PC817

Commit message: fix position
Parts:
- moved J28 5.46 mm to (89.0, 47.6), turned to 180 degrees
- moved J25 0.94 mm to (83.8, 143.1)
- moved J21 0.89 mm to (71.7, 143.1)
- moved J12 0.10 mm to (41.3, 143.1)
- moved J27 0.10 mm to (53.0, 143.1)
Routing:
- net OUT3_MT2: track 56.6 -> 59.0 mm
- net OUT4_MT2: track 58.4 -> 60.7 mm
- net OUT1_MT1: track 52.2 -> 53.1 mm
- net OUT2_MT1: track 61.9 -> 62.8 mm
Changed lines of the file:
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@@
   )
   (footprint "TerminalBlock_Phoenix:TerminalBlock_Phoenix_MKDS-1,5-2_1x02_P5.00mm_Horizontal" (layer "F.Cu")
-    (at 71.6934 142.2148)
+    (at 71.6934 143.1038)
     (descr "Terminal Block Phoenix MKDS-1,5-2, 2 pins, pitch 5mm, size 10x9.8mm^2, drill diamater 1.3mm, pad diameter 2.6mm, see http://www.farnell.com/datasheets/100425.pdf, script-generated using https://github.com/pointhi/kicad-footprint-generator/scripts/TerminalBlock_Phoenix")
     (tags "THT Terminal Block Phoenix MKDS-1,5-2 pitch 5mm size 10x9.8mm^2 drill 1.3mm pad 2.6mm")
@@
   )
   (footprint "TerminalBlock_Phoenix:TerminalBlock_Phoenix_MKDS-1,5-2_1x02_P5.00mm_Horizontal" (layer "F.Cu")
-    (at 83.5806 48.184)
+    (at 89.0124 47.5994 180)
     (descr "Terminal Block Phoenix MKDS-1,5-2, 2 pins, pitch 5mm, size 10x9.8mm^2, drill diamater 1.3mm, pad diameter 2.6mm, see http://www.farnell.com/datasheets/100425.pdf, script-generated using https://github.com/pointhi/kicad-footprint-generator/scripts/TerminalBlock_Phoenix")
     (tags "THT Terminal Block Phoenix MKDS-1,5-2 pitch 5mm size 10x9.8mm^2 drill 1.3mm pad 2.6mm")
@@
     (fp_circle (center 5 0) (end 6.5 0) (layer "F.Fab") (width 0.1) (fill none))
     (fp_circle (center 0 0) (end 1.5 0) (layer "F.Fab") (width 0.1) (fill none))
-    (pad "1" thru_hole rect (at 0 0) (size 2.6 2.6) (drill 1.3) (layers *.Cu *.Mask)
+    (pad "1" thru_hole rect (at 0 0 180) (size 2.6 2.6) (drill 1.3) (layers *.Cu *.Mask)
       (net 115 "unconnected-(J28-Pad1)") (pinfunction "Pin_1") (pintype "passive"))
-    (pad "2" thru_hole circle (at 5 0) (size 2.6 2.6) (drill 1.3) (layers *.Cu *.Mask)
+    (pad "2" thru_hole circle (at 5 0 180) (size 2.6 2.6) (drill 1.3) (layers *.Cu *.Mask)
       (net 116 "unconnected-(J28-Pad2)") (pinfunction "Pin_2") (pintype "passive"))
     (model "${KICAD6_3DMODEL_DIR}/TerminalBlock_Phoenix.3dshapes/TerminalBlock_Phoenix_MKDS-1,5-2_1x02_P5.00mm_Horizontal.wrl"
@@
   )
   (footprint "TerminalBlock_Phoenix:TerminalBlock_Phoenix_MKDS-1,5-2_1x02_P5.00mm_Horizontal" (layer "F.Cu")
-    (at 41.315 143.0022)
+    (at 41.315 143.1038)
     (descr "Terminal Block Phoenix MKDS-1,5-2, 2 pins, pitch 5mm, size 10x9.8mm^2, drill diamater 1.3mm, pad diameter 2.6mm, see http://www.farnell.com/datasheets/100425.pdf, script-generated using https://github.com/pointhi/kicad-footprint-generator/scripts/TerminalBlock_Phoenix")
     (tags "THT Terminal Block Phoenix MKDS-1,5-2 pitch 5mm size 10x9.8mm^2 drill 1.3mm pad 2.6mm")
@@
   )
   (footprint "TerminalBlock_Phoenix:TerminalBlock_Phoenix_MKDS-1,5-2_1x02_P5.00mm_Horizontal" (layer "F.Cu")
-    (at 83.8346 142.164)
+    (at 83.8346 143.1038)
     (descr "Terminal Block Phoenix MKDS-1,5-2, 2 pins, pitch 5mm, size 10x9.8mm^2, drill diamater 1.3mm, pad diameter 2.6mm, see http://www.farnell.com/datasheets/100425.pdf, script-generated using https://github.com/pointhi/kicad-footprint-generator/scripts/TerminalBlock_Phoenix")
     (tags "THT Terminal Block Phoenix MKDS-1,5-2 pitch 5mm size 10x9.8mm^2 drill 1.3mm pad 2.6mm")
@@
   )
   (footprint "TerminalBlock_Phoenix:TerminalBlock_Phoenix_MKDS-1,5-2_1x02_P5.00mm_Horizontal" (layer "F.Cu")
-    (at 53.0244 143.0022)
+    (at 53.0244 143.1038)
     (descr "Terminal Block Phoenix MKDS-1,5-2, 2 pins, pitch 5mm, size 10x9.8mm^2, drill diamater 1.3mm, pad diameter 2.6mm, see http://www.farnell.com/datasheets/100425.pdf, script-generated using https://github.com/pointhi/kicad-footprint-generator/scripts/TerminalBlock_Phoenix")
     (tags "THT Terminal Block Phoenix MKDS-1,5-2 pitch 5mm size 10x9.8mm^2 drill 1.3mm pad 2.6mm")
@@
   (segment (start 77.072066 142.847466) (end 77.0998 142.8752) (width 1) (layer "F.Cu") (net 8))
   (segment (start 66.421 125.984) (end 66.421 124.2568) (width 1) (layer "F.Cu") (net 8))
-  (segment (start 76.6934 142.2148) (end 76.6934 126.362666) (width 1) (layer "F.Cu") (net 8))
+  (segment (start 77.072066 125.984) (end 76.6934 126.362666) (width 1) (layer "F.Cu") (net 8))
+  (segment (start 76.6934 126.362666) (end 76.6934 143.1038) (width 1) (layer "F.Cu") (net 8))
   (segment (start 71.5942 103.6878) (end 74.4982 106.5918) (width 1) (layer "F.Cu") (net 8))
   (segment (start 74.4982 106.5918) (end 74.4982 122.9868) (width 1) (layer "F.Cu") (net 8))
-  (segment (start 76.6934 126.362666) (end 77.072066 125.984) (width 1) (layer "F.Cu") (net 8))
   (segment (start 71.6788 126.051733) (end 71.746533 125.984) (width 1) (layer "F.Cu") (net 9))
-  (segment (start 71.6934 126.037133) (end 71.746533 125.984) (width 1) (layer "F.Cu") (net 9))
+  (segment (start 71.746533 125.984) (end 71.6934 126.037133) (width 1) (layer "F.Cu") (net 9))
   (segment (start 72.0998 142.8752) (end 71.6788 142.4542) (width 1) (layer "F.Cu") (net 9))
-  (segment (start 71.6934 142.2148) (end 71.6934 126.037133) (width 1) (layer "F.Cu") (net 9))
+  (segment (start 71.6934 126.037133) (end 71.6934 143.1038) (width 1) (layer "F.Cu") (net 9))
   (segment (start 73.2028 129.54) (end 74.549 129.54) (width 1) (layer "B.Cu") (net 9))
   (segment (start 76.6742 102.4178) (end 75.401408 102.4178) (width 1) (layer "B.Cu") (net 9))
@@
   (segment (start 39.2514 89.2506) (end 40.798658 89.2506) (width 1) (layer "B.Cu") (net 13))
   (segment (start 39.2514 101.9506) (end 39.2514 102.227858) (width 1) (layer "F.Cu") (net 14))
-  (segment (start 46.99 125.9586) (end 46.99 142.3272) (width 1) (layer "F.Cu") (net 14))
+  (segment (start 46.99 125.9586) (end 46.99 141.0208) (width 1) (layer "F.Cu") (net 14))
   (segment (start 44.4754 122.7582) (end 44.5516 122.8344) (width 1) (layer "F.Cu") (net 14))
+  (segment (start 46.99 142.4288) (end 46.315 143.1038) (width 1) (layer "F.Cu") (net 14))
   (segment (start 44.4754 107.451858) (end 44.4754 122.7582) (width 1) (layer "F.Cu") (net 14))
   (segment (start 45.8216 122.8344) (end 46.99 124.0028) (width 1) (layer "F.Cu") (net 14))
@@
   (segment (start 36.7538 122.8344) (end 44.5516 122.8344) (width 1) (layer "F.Cu") (net 14))
   (segment (start 46.99 142.3272) (end 46.315 143.0022) (width 1) (layer "F.Cu") (net 14))
+  (segment (start 46.99 141.0208) (end 46.99 142.4288) (width 1) (layer "F.Cu") (net 14))
   (segment (start 39.2514 102.227858) (end 44.4754 107.451858) (width 1) (layer "F.Cu") (net 14))
-  (segment (start 41.402 125.9586) (end 41.402 142.9152) (width 1) (layer "F.Cu") (net 15))
+  (segment (start 46.99 141.0208) (end 46.99 142.3272) (width 1) (layer "F.Cu") (net 14))
+  (segment (start 41.402 140.7922) (end 41.402 143.0168) (width 1) (layer "F.Cu") (net 15))
+  (segment (start 41.402 125.9586) (end 41.402 140.7922) (width 1) (layer "F.Cu") (net 15))
+  (segment (start 41.402 140.7922) (end 41.402 142.9152) (width 1) (layer "F.Cu") (net 15))
   (segment (start 41.402 142.9152) (end 41.315 143.0022) (width 1) (layer "F.Cu") (net 15))
+  (segment (start 41.402 143.0168) (end 41.315 143.1038) (width 1) (layer "F.Cu") (net 15))
   (segment (start 41.402 125.9586) (end 41.402 128.2954) (width 1) (layer "B.Cu") (net 15))
   (segment (start 42.926 129.8194) (end 51.4604 129.8194) (width 1) (layer "B.Cu") (net 15))
